Commit message: feat: adapted to dual arm

File: kortex_description/multiple_robots/kortex_dual_robots.xacro (robot description, xacro)
@@ -19,5 +19,5 @@
         <parent link="world" />
         <!-- Here you can change the origin of the left arm-->
-        <origin xyz="-1 0 0" rpy="0 0 0" />
+        <origin xyz="0 0.66 0" rpy="0 0 0" />
     </joint>
     <joint name="world_to_$(arg right_prefix)root" type="fixed">
@@ -25,5 +25,5 @@
         <parent link="world" />
         <!-- Here you can change the origin of the right arm -->
-        <origin xyz="1 0 0" rpy="0 0 0" />
+        <origin xyz="0 0 0" rpy="0 0 0" />
     </joint>
     <xacro:load_robot
